File: 코네네.kicad_sch (KiCad schematic)
At the start: 46 parts, among them SW1 SW_Push, SW10 SW_Push, SW11 SW_Push, SW12 SW_Push, SW13 SW_Push, SW14 SW_Push, SW15 SW_Push, SW16 SW_Push, SW17 SW_Push, SW18 SW_Push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

Commit message: 왼쪽 판때기를 만들어따
Parts:
- added BT2: Battery_Cell, Connector_AMASS:AMASS_XT30U-M_1x02_P5.0mm_Vertical, symbol Device:Battery_Cell
- added D16, D20, D24, D25, D26, D27, D28, D29, D30, D31, D32, D33, D34, D35, D36, D37, D38, D39, D40, D41, D42: D, Diode_SMD:D_SOD-123, symbol Device:D
- added SW24, SW25, SW26, SW27, SW29, SW30, SW31, SW32, SW34, SW35, SW36, SW37, SW38, SW39, SW40, SW41, SW42, SW43, SW44, SW45, SW46: SW_Push, Library:Kailh_socket_PG1350, symbol Switch:SW_Push
- added SW28, SW33: SW_Push, Button_Switch_THT:SW_PUSH_1P1T_6x3.5mm_H4.3_APEM_MJTP1243, symbol Switch:SW_Push
- added U2: ~, Library:esp32_displaykit_s3, symbol New_Library:esp32_display_kit
Connections:
- net +BATT: now also BT2.1 (+), U2.2 (BAT)
- net GND: now also BT2.2 (-), SW28.2, SW33.2, U2.3 (GND)
- net boot: now also SW28.1, U2.26 (BOOT)
- net col1: now also SW24.2, SW25.2, SW26.2, SW27.2, U2.23 (GPIO35)
- net col2: now also SW29.2, SW30.2, SW31.2, SW32.2, U2.22 (GPIO36)
- net col3: now also SW34.2, SW35.2, SW36.2, SW37.2, U2.21 (GPIO37)
- net col4: now also SW38.2, SW39.2, SW40.2, U2.20 (GPIO38)
- net col5: now also SW41.2, SW42.2, SW43.2, U2.19 (GPIO39)
- net col6: now also SW44.2, SW45.2, SW46.2, U2.18 (GPIO40)
- net res: now also SW33.1, U2.1 (RES)
- net row1: now also D16.1 (K), D26.1 (K), D30.1 (K), D34.1 (K), D37.1 (K), D40.1 (K), U2.4 (GPIO8)
- net row2: now also D20.1 (K), D27.1 (K), D31.1 (K), D35.1 (K), D38.1 (K), D41.1 (K), U2.5 (GPIO7)
- net row3: now also D24.1 (K), D28.1 (K), D32.1 (K), D36.1 (K), D39.1 (K), D42.1 (K), U2.6 (GPIO6)
- net row4: now also D25.1 (K), D29.1 (K), D33.1 (K), U2.7 (GPIO5)
- new net: D24.2 (A), SW26.1
- new net: D37.2 (A), SW41.1
- new net: D41.2 (A), SW45.1
- new net: D36.2 (A), SW40.1
- new net: D31.2 (A), SW35.1
- new net: D29.2 (A), SW32.1
- new net: D16.2 (A), SW24.1
- new net: D42.2 (A), SW46.1
- new net: D25.2 (A), SW27.1
- new net: D35.2 (A), SW39.1
- new net: D39.2 (A), SW43.1
- new net: D30.2 (A), SW34.1
- new net: D40.2 (A), SW44.1
- new net: D32.2 (A), SW36.1
- new net: D33.2 (A), SW37.1
- new net: D38.2 (A), SW42.1
- new net: D27.2 (A), SW30.1
- new net: D20.2 (A), SW25.1
- new net: D28.2 (A), SW31.1
- new net: D34.2 (A), SW38.1
- new net: D26.2 (A), SW29.1
- no-connect marks 12 -> 24
Other:
- moved on the sheet: BT1, D1, D10, D11, D12, D13, D14, D15, D17, D18, D19, D2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
