File: 코네네.kicad_pcb (KiCad board)
At the start: 2 copper layers, 141.5 x 95.7 mm, 46 parts, among them SW1 SW_Push, SW10 SW_Push, SW11 SW_Push, SW12 SW_Push, SW13 SW_Push, SW14 SW_Push, SW15 SW_Push, SW16 SW_Push, SW17 SW_Push, SW18 SW_Push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

Commit message: 왼쪽 판때기를 만들어따
Parts:
- added BT2: Battery_Cell, Connector_AMASS:AMASS_XT30U-M_1x02_P5.0mm_Vertical, F.Cu at (155.5, 97.6)
- added D16: D, Diode_SMD:D_SOD-123, B.Cu at (134.9, 58.3)
- added D20: D, Diode_SMD:D_SOD-123, B.Cu at (135.0, 77.4)
- added D24: D, Diode_SMD:D_SOD-123, B.Cu at (135.0, 96.5)
- added D25: D, Diode_SMD:D_SOD-123, B.Cu at (149.5, 128.2)
- added D26: D, Diode_SMD:D_SOD-123, B.Cu at (116.0, 55.9)
- added D27: D, Diode_SMD:D_SOD-123, B.Cu at (115.8, 74.9)
- added D28: D, Diode_SMD:D_SOD-123, B.Cu at (115.9, 94.0)
- added D29: D, Diode_SMD:D_SOD-123, B.Cu at (127.3, 119.3)
- added D30: D, Diode_SMD:D_SOD-123, B.Cu at (96.9, 54.8)
- added D31: D, Diode_SMD:D_SOD-123, B.Cu at (96.8, 73.7)
- added D32: D, Diode_SMD:D_SOD-123, B.Cu at (96.8, 92.9)
- added D33: D, Diode_SMD:D_SOD-123, B.Cu at (103.3, 116.3)
- added D34: D, Diode_SMD:D_SOD-123, B.Cu at (77.7, 55.8)
- added D35: D, Diode_SMD:D_SOD-123, B.Cu at (77.7, 74.8)
- added D36: D, Diode_SMD:D_SOD-123, B.Cu at (77.8, 94.0)
- added D37: D, Diode_SMD:D_SOD-123, B.Cu at (58.8, 60.2)
- added D38: D, Diode_SMD:D_SOD-123, B.Cu at (58.8, 79.3)
- added D39: D, Diode_SMD:D_SOD-123, B.Cu at (58.7, 98.3)
- added D40: D, Diode_SMD:D_SOD-123, B.Cu at (39.8, 60.2)
- added D41: D, Diode_SMD:D_SOD-123, B.Cu at (39.6, 79.2)
- added D42: D, Diode_SMD:D_SOD-123, B.Cu at (39.7, 98.3)
- added SW24: SW_Push, Library:Kailh_socket_PG1350, F.Cu at (135.0, 63.0)
- added SW25: SW_Push, Library:Kailh_socket_PG1350, F.Cu at (135.0, 82.0)
- added SW26: SW_Push, Library:Kailh_socket_PG1350, F.Cu at (135.0, 101.1)
- added SW27: SW_Push, Library:Kailh_socket_PG1350, F.Cu at (146.9, 132.5)
- added SW28: SW_Push, Button_Switch_THT:SW_PUSH_1P1T_6x3.5mm_H4.3_APEM_MJTP1243, F.Cu at (159.3, 113.2)
- added SW29: SW_Push, Library:Kailh_socket_PG1350, F.Cu at (116.0, 60.6)
- added SW30: SW_Push, Library:Kailh_socket_PG1350, F.Cu at (116.0, 79.6)
- added SW31: SW_Push, Library:Kailh_socket_PG1350, F.Cu at (116.0, 98.7)
- added SW32: SW_Push, Library:Kailh_socket_PG1350, F.Cu at (125.9, 123.8)
- added SW33: SW_Push, Button_Switch_THT:SW_PUSH_1P1T_6x3.5mm_H4.3_APEM_MJTP1243, F.Cu at (149.3, 113.1)
- added SW34: SW_Push, Library:Kailh_socket_PG1350, F.Cu at (96.9, 59.4)
- added SW35: SW_Push, Library:Kailh_socket_PG1350, F.Cu at (96.9, 78.4)
- added SW36: SW_Push, Library:Kailh_socket_PG1350, F.Cu at (96.9, 97.5)
- added SW37: SW_Push, Library:Kailh_socket_PG1350, F.Cu at (103.3, 120.9)
- added SW38: SW_Push, Library:Kailh_socket_PG1350, F.Cu at (77.9, 60.6)
- added SW39: SW_Push, Library:Kailh_socket_PG1350, F.Cu at (77.9, 79.6)
- added SW40: SW_Push, Library:Kailh_socket_PG1350, F.Cu at (77.9, 98.7)
- added SW41: SW_Push, Library:Kailh_socket_PG1350, F.Cu at (58.8, 64.9)
- added SW42: SW_Push, Library:Kailh_socket_PG1350, F.Cu at (58.8, 83.9)
- added SW43: SW_Push, Library:Kailh_socket_PG1350, F.Cu at (58.8, 103.0)
- added SW44: SW_Push, Library:Kailh_socket_PG1350, F.Cu at (39.8, 64.9)
- added SW45: SW_Push, Library:Kailh_socket_PG1350, F.Cu at (39.8, 83.9)
- added SW46: SW_Push, Library:Kailh_socket_PG1350, F.Cu at (39.8, 103.0)
- added U2: ~, Library:esp32_displaykit_s3, F.Cu at (158.5, 108.8)
- moved BT1 137.8 mm to (191.2, 97.6)
- moved D1 137.8 mm to (217.5, 58.3)
- moved D10 137.8 mm to (255.6, 73.8)
- moved D11 137.8 mm to (255.6, 92.9)
- moved D12 137.8 mm to (249.1, 116.3)
- moved D13 137.8 mm to (274.6, 55.9)
- moved D14 137.8 mm to (274.6, 75.0)
- moved D15 137.8 mm to (274.6, 94.1)
- moved D2 137.8 mm to (217.5, 77.4)
- moved D21 137.8 mm to (312.9, 60.3)
- moved D23 137.8 mm to (312.8, 98.2)
- moved D3 137.8 mm to (217.4, 96.6)
- moved D4 137.8 mm to (203.2, 128.5)
- moved D5 137.8 mm to (236.6, 55.9)
- moved D6 137.8 mm to (236.6, 75.0)
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Routing:
- net col6: track 182.4 -> 388.8 mm, vias 2 -> 4
- net col5: track 155.6 -> 330.0 mm, vias 6 -> 8
- net col3: track 151.9 -> 310.0 mm, vias 6 -> 8
- net col4: track 131.0 -> 280.8 mm, vias 6 -> 8
- net row2: track 145.0 -> 294.7 mm, vias 2 -> 12
- net row1: track 153.1 -> 301.6 mm
- net col2: track 138.5 -> 286.1 mm, vias 6 -> 8
- net row3: track 139.1 -> 286.2 mm, vias 2 -> 12
- net col1: track 86.1 -> 206.7 mm, vias 0 -> 2
- net row4: track 115.7 -> 202.7 mm, vias 2 -> 6
- net GND: track 69.8 -> 141.4 mm, vias 1 -> 2
- net res: track 63.4 -> 125.9 mm
- net boot: track 65.9 -> 125.2 mm
- net +BATT: track 52.8 -> 92.9 mm
- net Net-(D25-A): track 0.00 -> 11.9 mm
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Other:
- board size 141.5 x 95.7 mm -> 292.1 x 95.7 mm

Commit message: 규멍을 뜌러따
Parts:
- added REF**: MountingHole_3.5mm, MountingHole:MountingHole_3.5mm, F.Cu at (141.6, 117.2)
- added REF**: MountingHole_3.5mm, MountingHole:MountingHole_3.5mm, B.Cu at (210.9, 117.2)
- added REF**: MountingHole_3.5mm, MountingHole:MountingHole_3.5mm, F.Cu at (125.0, 70.0)
- added REF**: MountingHole_3.5mm, MountingHole:MountingHole_3.5mm, F.Cu at (68.4, 71.8)
- added REF**: MountingHole_3.5mm, MountingHole:MountingHole_3.5mm, F.Cu at (104.4, 109.0)
- added REF**: MountingHole_3.5mm, MountingHole:MountingHole_3.5mm, F.Cu at (49.2, 93.4)
- added REF**: MountingHole_3.5mm, MountingHole:MountingHole_3.5mm, B.Cu at (303.3, 93.4)
- added REF**: MountingHole_3.5mm, MountingHole:MountingHole_3.5mm, B.Cu at (284.1, 71.8)
- added REF**: MountingHole_3.5mm, MountingHole:MountingHole_3.5mm, B.Cu at (227.5, 70.0)
- added REF**: MountingHole_3.5mm, MountingHole:MountingHole_3.5mm, B.Cu at (248.1, 109.0)
Routing:
- net GND: track 141.4 -> 250.9 mm, vias 2 -> 24
- net col2: track 286.1 -> 288.8 mm
- net col5: track 330.0 -> 332.7 mm
- net col4: track 280.8 -> 282.8 mm
- net col6: track 388.8 -> 390.6 mm
- net col1: track 206.7 -> 207.8 mm
- net col3: track 310.0 -> 310.8 mm
Other:
- outline, holes or cut-outs redrawn
